Commit message: Demo 2

File: workcell2_support/urdf/workcell.xacro (robot description, xacro)
@@ -29,5 +29,5 @@
     <origin xyz="0 0 0" rpy="0 0 0"/>
     <axis xyz="1 0 0"/>
-    <limit lower="0" upper="2" effort="0" velocity="1.0"/>
+    <limit lower="-2" upper="2" effort="0" velocity="1.0"/>
   </joint>
   <joint name="rail_y" type="prismatic">
@@ -36,5 +36,5 @@
     <origin xyz="0 0 0" rpy="0 0 0"/>
     <axis xyz="0 1 0"/>
-    <limit lower="0" upper="2" effort="0" velocity="1.0"/>
+    <limit lower="-2" upper="2" effort="0" velocity="1.0"/>
   </joint>
   <joint name="carriage_to_robot" type="fixed">
