Commit message: Semi working spooling demo; cylinders seem to have problems in tess

File: workcell4_support/urdf/workcell.xacro (robot description, xacro)
@@ -14,10 +14,10 @@
     <visual>
       <geometry>
-        <cylinder radius="0.25" length="0.75"/>
+        <mesh filename="package://workcell4_support/meshes/visual/cyl.stl"/>
       </geometry>
     </visual>
     <collision>
       <geometry>
-        <cylinder radius="0.5" length="0.5"/>
+        <mesh filename="package://workcell4_support/meshes/visual/cyl.stl"/>
       </geometry>
     </collision>
@@ -44,5 +44,5 @@
     <origin xyz="0 0 0" rpy="0 0 0"/>
     <axis xyz="0 0 1"/>
-    <limit lower="-3.14159" upper="3.14159" effort="0" velocity="1.0"/>
+    <limit lower="${-pi * 2}" upper="${pi * 2}" effort="0" velocity="1.0"/>
   </joint>
 </robot>
